Commit message: ok

File: BIG_BRAIN/src/robot/description/urdf/properties.urdf.xacro (robot description, xacro)
@@ -29,5 +29,5 @@
   <xacro:property name="tof_width" value="0.015"/>
   <xacro:property name="tof_height" value="0.01"/>
-  <xacro:property name="tof_z_offset" value="0.01"/> <!-- TOF center to camera bottom -->
+  <xacro:property name="tof_z_offset" value="0.0"/> <!-- TOF center to camera bottom -->
   <xacro:property name="tof_x_offset" value="0.006"/> <!-- TOF centor to camera center -->
   <!-- IMU -->
