Commit message: ok

File: BIG_BRAIN/src/robot/description/urdf/mobile_robot.xacro (robot description, xacro)
@@ -213,5 +213,5 @@
   <parent link="base_link"/>
   <child link="ultrasonic_right_link"/>
-  <origin xyz="${base_length/2 - ultrasonic_x_offset} ${-side_ultrasonic_y_offset} ${wheel_radius + wheel_z_offset - ultrasonic_z_offset}" rpy="0 0 0.05"/>
+  <origin xyz="${base_length/2 - ultrasonic_x_offset} ${-side_ultrasonic_y_offset} ${wheel_radius + wheel_z_offset - ultrasonic_z_offset}" rpy="0 0 ${-ultrasonic_z_angle}"/>
 </joint>
 <link name="ultrasonic_right_link">

Commit message: switch purpose

File: BIG_BRAIN/src/robot/description/urdf/mobile_robot.xacro (robot description, xacro)
@@ -148,11 +148,11 @@
   </link>
 <!-- ==================== Optical Frame ==================== -->
-<joint name="camera_depth_optical_joint" type="fixed">
+<joint name="camera_color_optical_joint" type="fixed">
   <parent link="camera_link"/>
-  <child link="camera_depth_optical_frame"/>
-  <!-- Pitch -90° to rotate X→forward, Y→down, Z→right (depth camera convention) -->
+  <child link="camera_color_optical_frame"/>
+  <!-- Standard ROS optical convention: Z forward, X right, Y down. -->
   <origin xyz="0 0 0" rpy="${-pi/2} 0 ${-pi/2}"/>
 </joint>
-<link name="camera_depth_optical_frame"/>
+<link name="camera_color_optical_frame"/>
 <!-- ==================== TOF ==================== -->
 <joint name="tof_joint" type="fixed">

Commit message: ok

File: BIG_BRAIN/src/robot/description/urdf/mobile_robot.xacro (robot description, xacro)
@@ -186,14 +186,14 @@
 </joint>
 <link name="imu_link"/>
-<!-- ==================== Ultrasonic Left ==================== -->
-<joint name="ultrasonic_left_joint" type="fixed">
-  <parent link="base_link"/>
-  <child link="ultrasonic_left_link"/>
-  <origin xyz="${base_length/2 - ultrasonic_x_offset} ${side_ultrasonic_y_offset} ${wheel_radius + wheel_z_offset - ultrasonic_z_offset}" rpy="0 0 ${ultrasonic_z_angle}"/>
-</joint>
-<link name="ultrasonic_left_link">
+<!-- ==================== Range Left ==================== -->
+<joint name="range_left_joint" type="fixed">
+  <parent link="base_link"/>
+  <child link="range_left_link"/>
+  <origin xyz="${base_length/2 - range_x_offset} ${side_range_y_offset} ${wheel_radius + wheel_z_offset - range_z_offset}" rpy="0 0 ${range_z_angle}"/>
+</joint>
+<link name="range_left_link">
   <visual>
     <origin xyz="0 0 0" rpy="0 0 0"/>
-    <geometry><box size="${ultrasonic_length} ${ultrasonic_width} ${ultrasonic_height}"/>
+    <geometry><box size="${range_length} ${range_width} ${range_height}"/>
     </geometry>
     <material name="green"/>
@@ -201,22 +201,22 @@
   <collision>
     <origin xyz="0 0 0" rpy="0 0 0"/>
-    <geometry><box size="${ultrasonic_length} ${ultrasonic_width} ${ultrasonic_height}"/>
+    <geometry><box size="${range_length} ${range_width} ${range_height}"/>
     </geometry>
   </collision>
   <inertial>
     <mass value="0.01"/>
-    <xacro:box_inertia mass="0.01" x="${ultrasonic_length}" y="${ultrasonic_width}" z="${ultrasonic_height}"/>
+    <xacro:box_inertia mass="0.01" x="${range_length}" y="${range_width}" z="${range_height}"/>
   </inertial>
 </link>
-<!-- ==================== Ultrasonic Right ==================== -->
-<joint name="ultrasonic_right_joint" type="fixed">
-  <parent link="base_link"/>
-  <child link="ultrasonic_right_link"/>
-  <origin xyz="${base_length/2 - ultrasonic_x_offset} ${-side_ultrasonic_y_offset} ${wheel_radius + wheel_z_offset - ultrasonic_z_offset}" rpy="0 0 ${-ultrasonic_z_angle}"/>
-</joint>
-<link name="ultrasonic_right_link">
+<!-- ==================== Range Right ==================== -->
+<joint name="range_right_joint" type="fixed">
+  <parent link="base_link"/>
+  <child link="range_right_link"/>
+  <origin xyz="${base_length/2 - range_x_offset} ${-side_range_y_offset} ${wheel_radius + wheel_z_offset - range_z_offset}" rpy="0 0 ${-range_z_angle}"/>
+</joint>
+<link name="range_right_link">
   <visual>
     <origin xyz="0 0 0" rpy="0 0 0"/>
-    <geometry><box size="${ultrasonic_length} ${ultrasonic_width} ${ultrasonic_height}"/>
+    <geometry><box size="${range_length} ${range_width} ${range_height}"/>
     </geometry>
     <material name="green"/>
@@ -224,10 +224,10 @@
   <collision>
     <origin xyz="0 0 0" rpy="0 0 0"/>
-    <geometry><box size="${ultrasonic_length} ${ultrasonic_width} ${ultrasonic_height}"/>
+    <geometry><box size="${range_length} ${range_width} ${range_height}"/>
     </geometry>
   </collision>
   <inertial>
     <mass value="0.01"/>
-    <xacro:box_inertia mass="0.01" x="${ultrasonic_length}" y="${ultrasonic_width}" z="${ultrasonic_height}"/>
+    <xacro:box_inertia mass="0.01" x="${range_length}" y="${range_width}" z="${range_height}"/>
   </inertial>
 </link>

File: BIG_BRAIN/src/robot/description/urdf/properties.urdf.xacro (robot description, xacro)
@@ -33,12 +33,12 @@
   <!-- IMU -->
   <xacro:property name="imu_z_offset" value="0.0"/> <!-- MPU to Base bottom -->
-  <!-- Ultrasonic -->
-  <xacro:property name="ultrasonic_x_offset" value="0.012"/> <!-- Ultrasonic center to Base front -->
-  <xacro:property name="side_ultrasonic_y_offset" value="0.105"/> <!-- Side ultrasonic center to Base center -->
-  <xacro:property name="ultrasonic_z_offset" value="0.012"/> <!-- Ultrasonic center to Base bottom -->
-  <xacro:property name="ultrasonic_z_angle" value="0.43"/> <!-- Side ultrasonic angle to Base front -->
-  <xacro:property name="ultrasonic_length" value="0.01"/>
-  <xacro:property name="ultrasonic_width" value="0.04"/>
-  <xacro:property name="ultrasonic_height" value="0.02"/>
+  <!-- Range -->
+  <xacro:property name="range_x_offset" value="0.019"/> <!-- Range center to Base front -->
+  <xacro:property name="side_range_y_offset" value="0.093"/> <!-- Side range center to Base center -->
+  <xacro:property name="range_z_offset" value="0.01"/> <!-- Range center to Base bottom -->
+  <xacro:property name="range_z_angle" value="0.3554"/> <!-- Side range angle to Base front -->
+  <xacro:property name="range_length" value="0.016"/>
+  <xacro:property name="range_width" value="0.005"/>
+  <xacro:property name="range_height" value="0.014"/>
   <!-- Materials -->
   <material name="blue">

Commit message: ok

File: BIG_BRAIN/src/robot/description/urdf/mobile_robot.xacro (robot description, xacro)
@@ -148,11 +148,11 @@
   </link>
 <!-- ==================== Optical Frame ==================== -->
-<joint name="camera_color_optical_joint" type="fixed">
+<joint name="camera_depth_optical_joint" type="fixed">
   <parent link="camera_link"/>
-  <child link="camera_color_optical_frame"/>
+  <child link="camera_depth_optical_frame"/>
   <!-- Standard ROS optical convention: Z forward, X right, Y down. -->
   <origin xyz="0 0 0" rpy="${-pi/2} 0 ${-pi/2}"/>
 </joint>
-<link name="camera_color_optical_frame"/>
+<link name="camera_depth_optical_frame"/>
 <!-- ==================== TOF ==================== -->
 <joint name="tof_joint" type="fixed">

Commit message: ok

File: BIG_BRAIN/src/robot/description/urdf/mobile_robot.xacro (robot description, xacro)
@@ -232,3 +232,27 @@
   </inertial>
 </link>
+<!-- ==================== RGB Camera ==================== -->
+<joint name="rgb_camera_joint" type="fixed">
+  <parent link="base_link"/>
+  <child link="rgb_camera_link"/>
+  <origin xyz="${base_length/2 - rgb_camera_x_offset} 0 ${wheel_radius + wheel_z_offset + base_height + rgb_camera_z_offset}" rpy="0 0 0"/>
+</joint>
+<link name='rgb_camera_link'>
+    <visual>
+      <origin xyz="${rgb_camera_length/2} 0 0" rpy="0 0 0"/>
+      <geometry><box size="${rgb_camera_length} ${rgb_camera_width} ${rgb_camera_height}"/>
+      </geometry>
+      <material name="green"/>
+    </visual>
+    <collision>
+      <origin xyz="${rgb_camera_length/2} 0 0" rpy="0 0 0"/>
+      <geometry><box size="${rgb_camera_length} ${rgb_camera_width} ${rgb_camera_height}"/>
+      </geometry>
+    </collision>
+    <inertial>
+      <origin xyz="${rgb_camera_length/2} 0 0" rpy="0 0 0"/>
+      <mass value="0.01"/>
+      <xacro:box_inertia mass="0.01" x="${rgb_camera_length}" y="${rgb_camera_width}" z="${rgb_camera_height}"/>
+    </inertial>
+</link>
 </robot>

File: BIG_BRAIN/src/robot/description/urdf/properties.urdf.xacro (robot description, xacro)
@@ -25,4 +25,10 @@
   <xacro:property name="camera_z_offset" value="0.028"/> <!-- Camera upper to Base upper -->
   <xacro:property name="camera_x_offset" value="0.023"/> <!-- Camera front to Base front -->
+  <!-- RGB Camera -->
+  <xacro:property name="rgb_camera_length" value="0.01"/>
+  <xacro:property name="rgb_camera_width" value="0.036"/>
+  <xacro:property name="rgb_camera_height" value="0.036"/>
+  <xacro:property name="rgb_camera_z_offset" value="0.05"/> <!-- Camera center to Base upper -->
+  <xacro:property name="rgb_camera_x_offset" value="0.01"/> <!-- Camera center to Base front -->
   <!-- TOF -->
   <xacro:property name="tof_length" value="0.003"/>
